Commit message: changed camera position to 1m and callibrated

File: src/description/urdf/robot_base.xacro (robot description, xacro)
@@ -200,5 +200,5 @@
   <parent link="base_link"/>
   <child link="camera_link"/>
-  <origin xyz="0.15 0 2" rpy="0 0.4 0"/> <!-- chcanged camera and turret positions-->
+  <origin xyz="0.15 0 1" rpy="0 0.25 0"/> <!-- chcanged camera and turret positions-->
 </joint>
     <xacro:macro name="wheel" params="name x y">
